File: STX3Micro.brd (EAGLE design)
At the start: 82.2 x 45.7 mm, 6 parts, among them X1 LTI-SASF54GT

Commit message: Fixed Feed Point
Parts:
- added JP1: (no value), pinhead:1X02
- added Q1: BSS84, transistor-small-signal:SOT23
- added U1: ATTINY85-20SU, Atmel_By_element14_Batch_1-00:SOIC127P798X216-8N
- moved SV1 13.3 mm to (69.8, 30.5), turned to 180 degrees
- moved SV2 9.92 mm to (76.2, 58.4)
Connections:
- new net N$14: JP1.1, SV1.1, SV2.1, U$1.10, U$1.11, U$1.12, U$1.13, U$1.15, U$1.16, U$1.17, U$1.18, U$1.19, U$1.20, U$1.8, U$1.9, U1.4, X1.2, X1.3, X1.4, X1.5
- net N$1: now also SV1.5, U1.1; no longer SV1.1, U$1.2
- net N$12: now also U1.2
- net N$13: now also Q1.2
- net N$16: now also Q1.1, U1.7; no longer SV1.6, SV2.1, U$1.10, U$1.11, U$1.12, U$1.13, U$1.15, U$1.16, U$1.17, U$1.18, U$1.19, U$1.20, U$1.8, U$1.9, X1.2, X1.3, X1.4, X1.5
- net N$2: now also U1.3; no longer SV1.2
- net N$3: now also U1.5; no longer SV1.3
- net N$4: now also JP1.2, Q1.3, SV1.3, U1.8; no longer SV1.4
- net N$5: now also SV1.4, U1.6; no longer SV1.5, U$1.1
Routing:
- net N$16: track 93.2 -> 0.00 mm
- net N$14: track 0.00 -> 80.7 mm
- net N$5: track 36.5 -> 0.00 mm, vias 1 -> 0
- net N$1: track 33.2 -> 0.00 mm, vias 1 -> 0
- net N$2: track 28.8 -> 0.00 mm
- net N$4: track 45.5 -> 69.0 mm
- net N$3: track 20.7 -> 0.00 mm, vias 1 -> 0
- net N$13: track 21.7 -> 36.5 mm
- net N$11: track 21.5 -> 18.4 mm
- net N$12: track 35.4 -> 38.2 mm
- net N$8: track 15.8 -> 18.1 mm, vias 2 -> 0
- net N$10: track 22.5 -> 22.0 mm
- net N$6: track 29.7 -> 29.2 mm
- net N$9: track 26.1 -> 25.6 mm
Other:
- board size 82.2 x 45.7 mm -> 83.5 x 45.7 mm
- board text added: "STX3 Breakout with Controller"
- board text removed: "STX3 Breakout"

Commit message: Micro Board Routing Done
Routing:
- net N$14: track 80.7 -> 157.9 mm, vias 0 -> 2
- net N$16: track 0.00 -> 46.4 mm, vias 0 -> 2
- net N$5: track 0.00 -> 30.1 mm, vias 0 -> 2
- net N$1: track 0.00 -> 24.8 mm
- net N$3: track 0.00 -> 18.5 mm
- net N$2: track 0.00 -> 15.0 mm
- net N$12: track 38.2 -> 46.0 mm
- net N$10: track 22.0 -> 23.7 mm
- net N$4: track 69.0 -> 68.4 mm, vias 1 -> 2
- net N$8: track 18.1 -> 18.7 mm, vias 0 -> 2

Commit message: Fixed Ground Loop
Routing:
- net N$14: track 157.9 -> 149.6 mm
Changed lines of the file:
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@@
 <contactref element="JP1" pad="1"/>
 <contactref element="SV1" pad="1"/>
-<wire x1="68.58" y1="40.64" x2="68.58" y2="38.1" width="0.254" layer="1"/>
 <wire x1="73.66" y1="36.83" x2="71.12" y2="36.83" width="0.254" layer="1"/>
 <wire x1="73.66" y1="36.83" x2="76.2" y2="36.83" width="0.254" layer="1"/>
@@
 <wire x1="68.58" y1="52.07" x2="68.58" y2="50.8" width="0.254" layer="1"/>
 <wire x1="68.58" y1="50.8" x2="68.58" y2="48.26" width="0.254" layer="1"/>
-<wire x1="68.58" y1="52.07" x2="71.12" y2="54.61" width="0.254" layer="1"/>
+<wire x1="68.58" y1="52.07" x2="69.215" y2="52.705" width="0.254" layer="1"/>
 <wire x1="71.12" y1="55.88" x2="68.58" y2="58.42" width="0.254" layer="1"/>
 <wire x1="71.12" y1="54.61" x2="71.12" y2="55.88" width="0.254" layer="1"/>
@@
 <wire x1="68.58" y1="58.42" x2="67.31" y2="58.42" width="0.254" layer="16"/>
 <wire x1="64.77" y1="60.96" x2="64.77" y2="66.04" width="0.254" layer="1"/>
-<wire x1="71.12" y1="54.61" x2="71.12" y2="43.18" width="0.254" layer="1"/>
 <wire x1="81.28" y1="26.67" x2="81.28" y2="29.21" width="0.4064" layer="1"/>
-<wire x1="68.58" y1="40.64" x2="71.12" y2="40.64" width="0.4064" layer="1"/>
-<wire x1="71.12" y1="40.64" x2="71.12" y2="43.18" width="0.4064" layer="1"/>
 <wire x1="81.28" y1="29.21" x2="84.455" y2="29.21" width="0.4064" layer="1"/>
 <wire x1="84.455" y1="29.21" x2="84.455" y2="28.575" width="0.4064" layer="1"/>
@@
 <wire x1="59.69" y1="60.96" x2="64.77" y2="60.96" width="0.4064" layer="16"/>
 <wire x1="64.77" y1="60.96" x2="64.77" y2="46.355" width="0.4064" layer="16"/>
-<wire x1="64.77" y1="46.355" x2="48.895" y2="46.355" width="0.4064" layer="16"/>
-<wire x1="48.895" y1="46.355" x2="48.895" y2="38.1" width="0.4064" layer="16"/>
-<wire x1="48.895" y1="38.1" x2="64.77" y2="38.1" width="0.4064" layer="16"/>
+<wire x1="68.58" y1="40.64" x2="68.58" y2="38.1" width="0.4064" layer="1"/>
+<wire x1="68.58" y1="38.1" x2="64.77" y2="38.1" width="0.4064" layer="1"/>
 <via x="64.77" y="38.1" extent="1-16" drill="0.6"/>
-<wire x1="64.77" y1="38.1" x2="68.58" y2="38.1" width="0.4064" layer="1"/>
+<wire x1="64.77" y1="38.1" x2="48.895" y2="38.1" width="0.4064" layer="16"/>
+<wire x1="48.895" y1="38.1" x2="48.895" y2="46.355" width="0.4064" layer="16"/>
+<wire x1="48.895" y1="46.355" x2="64.77" y2="46.355" width="0.4064" layer="16"/>
 <via x="64.77" y="46.355" extent="1-16" drill="0.6"/>
 <wire x1="64.77" y1="46.355" x2="68.58" y2="46.355" width="0.4064" layer="1"/>
+<wire x1="68.58" y1="46.355" x2="68.58" y2="53.34" width="0.4064" layer="1"/>
+<wire x1="68.58" y1="53.34" x2="69.215" y2="53.34" width="0.4064" layer="1"/>
+<wire x1="69.215" y1="53.34" x2="69.215" y2="52.705" width="0.4064" layer="1"/>
+<wire x1="69.215" y1="52.705" x2="71.12" y2="54.61" width="0.4064" layer="1"/>
 </signal>
 <signal name="N$1">
