File: STX3Micro.brd (EAGLE design)
At the start: 83.5 x 45.7 mm, 9 parts, among them Q1 BSS84, U1 ATTINY85-20SU, X1 LTI-SASF54GT

Commit message: Fixed CTS/RTS Connections
Connections:
- new net N$17: SV1.6, U$1.2
- new net N$18: SV1.2, U$1.1
Routing:
- net N$18: track 0.00 -> 39.6 mm, vias 0 -> 2
- net N$17: track 0.00 -> 39.1 mm, vias 0 -> 1
Changed lines of the file:
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@@
 <wire x1="93.8784" y1="31.115" x2="95.25" y2="31.115" width="0.4064" layer="1"/>
+</signal>
+<signal name="N$17">
+<contactref element="U$1" pad="2"/>
+<contactref element="SV1" pad="6"/>
+<wire x1="86.36" y1="52.07" x2="88.9" y2="54.61" width="0.2032" layer="1"/>
+<wire x1="86.36" y1="45.72" x2="86.36" y2="52.07" width="0.2032" layer="1"/>
+<wire x1="76.2" y1="35.56" x2="86.36" y2="45.72" width="0.2032" layer="16"/>
+<wire x1="68.58" y1="35.56" x2="76.2" y2="35.56" width="0.2032" layer="16"/>
+<wire x1="63.5" y1="30.48" x2="68.58" y2="35.56" width="0.2032" layer="16"/>
+<via x="86.36" y="45.72" extent="1-16" drill="0.508"/>
+</signal>
+<signal name="N$18">
+<contactref element="U$1" pad="1"/>
+<contactref element="SV1" pad="2"/>
+<wire x1="88.9" y1="57.15" x2="91.44" y2="54.61" width="0.2032" layer="1"/>
+<wire x1="85.09" y1="57.15" x2="88.9" y2="57.15" width="0.2032" layer="1"/>
+<wire x1="85.09" y1="43.18" x2="85.09" y2="57.15" width="0.2032" layer="1"/>
+<wire x1="76.2" y1="34.29" x2="85.09" y2="43.18" width="0.2032" layer="16"/>
+<wire x1="74.93" y1="34.29" x2="76.2" y2="34.29" width="0.2032" layer="16"/>
+<wire x1="73.66" y1="33.02" x2="74.93" y2="34.29" width="0.2032" layer="1"/>
+<wire x1="73.66" y1="30.48" x2="73.66" y2="33.02" width="0.2032" layer="1"/>
+<via x="85.09" y="43.18" extent="1-16" drill="0.508"/>
+<via x="74.93" y="34.29" extent="1-16" drill="0.508"/>
 </signal>
 </signals>
